File: effectHardware/codec.kicad_sch (KiCad schematic)
At the start: 21 parts, among them IC1 LMP8350MA_NOPB, U12 ES9290, U13 74LVC1G04, U14 THS4551xRGT, Y1 XRCGB24M576F0G00R0

Commit message: added lib
Parts:
- C41, C63, C64, C65, C66, C67, C68, C69, C70, C71, C72, C73, C74, C75: symbol Device:C_Small -> Library:C_Small
- IC1: symbol LMP8350MA_NOPB:LMP8350MA_NOPB -> Library:LMP8350MA_NOPB
- R36, R37: symbol Device:R_Small -> Library:R_Small
- U12: symbol Audio:es9290 -> Library:es9290
- U13: symbol 74xGxx:74LVC1G04 -> Library:74LVC1G04
- U14: symbol Amplifier_Difference:THS4551xRGT -> Library:THS4551xRGT
- Y1: symbol XRCGB24M576F0G00R0:XRCGB24M576F0G00R0 -> Library:XRCGB24M576F0G00R0
Changed lines of the file:
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@@
 	)
 	(symbol
-		(lib_id "power:GND")
+		(lib_id "Library:GND")
 		(at 100.33 64.77 270)
 		(unit 1)
@@
 	)
 	(symbol
-		(lib_id "power:GND")
+		(lib_id "Library:GND")
 		(at 110.49 58.42 270)
 		(unit 1)
@@
 	)
 	(symbol
-		(lib_id "Device:R_Small")
+		(lib_id "Library:R_Small")
 		(at 135.89 78.74 0)
 		(unit 1)
@@
 	)
 	(symbol
-		(lib_id "power:GND")
+		(lib_id "Library:GND")
 		(at 130.81 31.75 180)
 		(unit 1)
@@
 	)
 	(symbol
-		(lib_id "power:GND")
+		(lib_id "Library:GND")
 		(at 143.51 57.15 90)
 		(unit 1)
@@
 	)
 	(symbol
-		(lib_id "Audio:es9290")
+		(lib_id "Library:es9290")
 		(at 123.19 52.07 0)
 		(unit 1)
@@
 	)
 	(symbol
-		(lib_id "power:GND")
+		(lib_id "Library:GND")
 		(at 135.89 50.8 180)
 		(unit 1)
@@
 	)
 	(symbol
-		(lib_id "74xGxx:74LVC1G04")
+		(lib_id "Library:74LVC1G04")
 		(at 149.86 104.14 180)
 		(unit 1)
@@
 	)
 	(symbol
-		(lib_id "Device:C_Small")
+		(lib_id "Library:C_Small")
 		(at 157.48 66.04 270)
 		(unit 1)
@@
 	)
 	(symbol
-		(lib_id "Device:C_Small")
+		(lib_id "Library:C_Small")
 		(at 129.54 35.56 0)
 		(unit 1)
@@
 	)
 	(symbol
-		(lib_id "Device:R_Small")
+		(lib_id "Library:R_Small")
 		(at 148.59 119.38 90)
 		(unit 1)
@@
 	)
 	(symbol
-		(lib_id "Device:C_Small")
+		(lib_id "Library:C_Small")
 		(at 173.99 104.14 0)
 		(unit 1)
@@
 	)
 	(symbol
-		(lib_id "power:GND")
+		(lib_id "Library:GND")
 		(at 154.94 93.98 180)
 		(unit 1)
@@
 	)
 	(symbol
-		(lib_id "power:GND")
+		(lib_id "Library:GND")
 		(at 132.08 45.72 180)
 		(unit 1)
@@
 	)
 	(symbol
-		(lib_id "Device:C_Small")
+		(lib_id "Library:C_Small")
 		(at 111.76 67.31 270)
 		(unit 1)
@@
 	)
 	(symbol
-		(lib_id "power:GND")
+		(lib_id "Library:GND")
 		(at 134.62 100.33 0)
 		(unit 1)
@@
 	)
 	(symbol
-		(lib_id "power:+3V3")
+		(lib_id "Library:+3V3")
 		(at 143.51 68.58 180)
 		(unit 1)
@@
 	)
 	(symbol
-		(lib_id "power:+3V3")
+		(lib_id "Library:+3V3")
 		(at 154.94 114.3 90)
 		(unit 1)
@@
 	)
 	(symbol
-		(lib_id "power:+3V3")
+		(lib_id "Library:+3V3")
 		(at 120.65 57.15 0)
 		(unit 1)
@@
 	)
 	(symbol
-		(lib_id "power:+3V3")
+		(lib_id "Library:+3V3")
 		(at 127 80.01 180)
 		(unit 1)
@@
 	)
 	(symbol
-		(lib_id "Device:C_Small")
+		(lib_id "Library:C_Small")
 		(at 134.62 97.79 0)
 		(unit 1)
@@
 	)
 	(symbol
-		(lib_id "Device:C_Small")
+		(lib_id "Library:C_Small")
 		(at 166.37 132.08 270)
 		(unit 1)
@@
 	)
 	(symbol
-		(lib_id "power:GND")
+		(lib_id "Library:GND")
 		(at 168.91 132.08 90)
 		(unit 1)
@@
 	)
 	(symbol
-		(lib_id "Device:C_Small")
+		(lib_id "Library:C_Small")
 		(at 118.11 57.15 270)
 		(unit 1)
@@
 	)
 	(symbol
-		(lib_id "LMP8350MA_NOPB:LMP8350MA_NOPB")
+		(lib_id "Library:LMP8350MA_NOPB")
 		(at 34.29 38.1 0)
 		(unit 1)
@@
 	)
 	(symbol
-		(lib_id "Amplifier_Difference:THS4551xRGT")
+		(lib_id "Library:THS4551xRGT")
 		(at 31.75 182.88 270)
 		(unit 2)
@@
 	)
 	(symbol
-		(lib_id "Device:C_Small")
+		(lib_id "Library:C_Small")
 		(at 118.11 68.58 270)
 		(unit 1)
@@
 	)
 	(symbol
-		(lib_id "Device:C_Small")
+		(lib_id "Library:C_Small")
 		(at 146.05 68.58 270)
 		(unit 1)
@@
 	)
 	(symbol
-		(lib_id "XRCGB24M576F0G00R0:XRCGB24M576F0G00R0")
+		(lib_id "Library:XRCGB24M576F0G00R0")
 		(at 130.81 132.08 0)
 		(unit 1)
@@
 	)
 	(symbol
-		(lib_id "power:GND")
+		(lib_id "Library:GND")
 		(at 135.89 85.09 0)
 		(unit 1)
@@
 	)
 	(symbol
-		(lib_id "Device:C_Small")
+		(lib_id "Library:C_Small")
 		(at 128.27 137.16 180)
 		(unit 1)
@@
 	)
 	(symbol
-		(lib_id "power:GND")
+		(lib_id "Library:GND")
 		(at 133.35 76.2 0)
 		(unit 1)
@@
 	)
 	(symbol
-		(lib_id "Device:C_Small")
+		(lib_id "Library:C_Small")
 		(at 113.03 58.42 270)
 		(unit 1)
@@
 	)
 	(symbol
-		(lib_id "Device:C_Small")
+		(lib_id "Library:C_Small")
 		(at 125.73 41.91 90)
 		(unit 1)
@@
 	)
 	(symbol
-		(lib_id "Device:C_Small")
+		(lib_id "Library:C_Small")
 		(at 124.46 77.47 270)
 		(unit 1)
@@
 	)
 	(symbol
-		(lib_id "power:GND")
+		(lib_id "Library:GND")
 		(at 167.64 67.31 90)
 		(unit 1)
@@
 	)
 	(symbol
-		(lib_id "Device:C_Small")
+		(lib_id "Library:C_Small")
 		(at 104.14 66.04 270)
 		(unit 1)
@@
 	)
 	(symbol
-		(lib_id "power:GND")
+		(lib_id "Library:GND")
 		(at 128.27 139.7 0)
 		(unit 1)
