File: effectHardware/effect_pwr.kicad_sch (KiCad schematic)
At the start: 26 parts, among them J2 Conn_02x05_Odd_Even, U3 LM1117DT-5.0, U4 ADP150AUJZ-3.3-R7

Commit message: added lib
Parts:
- C1, C10, C11, C12, C2, C3, C4, C5, C6, C7, C8, C9: symbol Device:C -> Library:C
- D1, D2: symbol Device:D -> Library:D
- D3, D4, D5, D6: symbol Device:LED -> Library:LED
- J2: symbol Connector_Generic:Conn_02x05_Odd_Even -> Library:Conn_02x05_Odd_Even
- L2: symbol Device:L -> Library:L
- R1, R2, R3, R4: symbol Device:R -> Library:R
- U3: symbol Regulator_Linear:LM1117DT-5.0 -> Library:LM1117DT-5.0
- U4: symbol ADP150AUJZ-2.0-R7:ADP150AUJZ-2.0-R7 -> Library:ADP150AUJZ-2.0-R7
Changed lines of the file:
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@@
 	)
 	(symbol
-		(lib_id "power:GND")
+		(lib_id "Library:GND")
 		(at 83.82 82.55 0)
 		(mirror y)
@@
 	)
 	(symbol
-		(lib_id "Device:C")
+		(lib_id "Library:C")
 		(at 142.24 85.09 0)
 		(unit 1)
@@
 	)
 	(symbol
-		(lib_id "Device:R")
+		(lib_id "Library:R")
 		(at 167.64 97.79 90)
 		(unit 1)
@@
 	)
 	(symbol
-		(lib_id "power:GND")
+		(lib_id "Library:GND")
 		(at 179.07 106.68 90)
 		(unit 1)
@@
 	)
 	(symbol
-		(lib_id "power:+12V")
+		(lib_id "Library:+12V")
 		(at 163.83 106.68 90)
 		(unit 1)
@@
 	)
 	(symbol
-		(lib_id "Device:LED")
+		(lib_id "Library:LED")
 		(at 175.26 97.79 0)
 		(mirror x)
@@
 	)
 	(symbol
-		(lib_id "Device:C")
+		(lib_id "Library:C")
 		(at 111.76 91.44 0)
 		(unit 1)
@@
 	)
 	(symbol
-		(lib_id "Device:D")
+		(lib_id "Library:D")
 		(at 107.95 77.47 180)
 		(unit 1)
@@
 	)
 	(symbol
-		(lib_id "power:GND")
+		(lib_id "Library:GND")
 		(at 142.24 92.71 90)
 		(unit 1)
@@
 	)
 	(symbol
-		(lib_id "power:GND")
+		(lib_id "Library:GND")
 		(at 146.05 97.79 90)
 		(unit 1)
@@
 	)
 	(symbol
-		(lib_id "Connector_Generic:Conn_02x05_Odd_Even")
+		(lib_id "Library:Conn_02x05_Odd_Even")
 		(at 96.52 82.55 0)
 		(mirror x)
@@
 	)
 	(symbol
-		(lib_id "Device:C")
+		(lib_id "Library:C")
 		(at 179.07 67.31 0)
 		(unit 1)
@@
 	)
 	(symbol
-		(lib_id "Device:L")
+		(lib_id "Library:L")
 		(at 128.27 50.8 270)
 		(unit 1)
@@
 	)
 	(symbol
-		(lib_id "power:+5V")
+		(lib_id "Library:+5V")
 		(at 130.81 97.79 90)
 		(unit 1)
@@
 	)
 	(symbol
-		(lib_id "power:+12V")
+		(lib_id "Library:+12V")
 		(at 111.76 80.01 270)
 		(unit 1)
@@
 	)
 	(symbol
-		(lib_id "Device:LED")
+		(lib_id "Library:LED")
 		(at 142.24 97.79 180)
 		(unit 1)
@@
 	)
 	(symbol
-		(lib_id "Device:C")
+		(lib_id "Library:C")
 		(at 110.49 54.61 0)
 		(unit 1)
@@
 	)
 	(symbol
-		(lib_id "Device:C")
+		(lib_id "Library:C")
 		(at 147.32 67.31 0)
 		(unit 1)
@@
 	)
 	(symbol
-		(lib_id "Device:R")
+		(lib_id "Library:R")
 		(at 167.64 106.68 90)
 		(unit 1)
@@
 	)
 	(symbol
-		(lib_id "power:GND")
+		(lib_id "Library:GND")
 		(at 146.05 105.41 90)
 		(unit 1)
@@
 	)
 	(symbol
-		(lib_id "Device:D")
+		(lib_id "Library:D")
 		(at 107.95 87.63 0)
 		(unit 1)
@@
 	)
 	(symbol
-		(lib_id "Device:C")
+		(lib_id "Library:C")
 		(at 153.67 85.09 0)
 		(unit 1)
@@
 	)
 	(symbol
-		(lib_id "Device:C")
+		(lib_id "Library:C")
 		(at 90.17 54.61 0)
 		(mirror y)
@@
 	)
 	(symbol
-		(lib_id "power:+12V")
+		(lib_id "Library:+12V")
 		(at 142.24 81.28 0)
 		(unit 1)
@@
 	)
 	(symbol
-		(lib_id "Device:C")
+		(lib_id "Library:C")
 		(at 111.76 72.39 0)
 		(unit 1)
@@
 	)
 	(symbol
-		(lib_id "power:+3.3V")
+		(lib_id "Library:+3.3V")
 		(at 130.81 105.41 90)
 		(unit 1)
@@
 	)
 	(symbol
-		(lib_id "power:-12V")
+		(lib_id "Library:-12V")
 		(at 166.37 81.28 0)
 		(unit 1)
@@
 	)
 	(symbol
-		(lib_id "Device:LED")
+		(lib_id "Library:LED")
 		(at 175.26 106.68 180)
 		(unit 1)
@@
 	)
 	(symbol
-		(lib_id "power:GND")
+		(lib_id "Library:GND")
 		(at 100.33 60.96 0)
 		(unit 1)
@@
 	)
 	(symbol
-		(lib_id "Device:R")
+		(lib_id "Library:R")
 		(at 134.62 105.41 90)
 		(unit 1)
@@
 	)
 	(symbol
-		(lib_id "Device:C")
+		(lib_id "Library:C")
 		(at 166.37 85.09 0)
 		(unit 1)
@@
 	)
 	(symbol
-		(lib_id "power:+3.3V")
+		(lib_id "Library:+3.3V")
 		(at 175.26 45.72 0)
 		(unit 1)
@@
 	)
 	(symbol
-		(lib_id "Device:C")
+		(lib_id "Library:C")
 		(at 142.24 67.31 0)
 		(mirror y)
@@
 	)
 	(symbol
-		(lib_id "power:+5V")
+		(lib_id "Library:+5V")
 		(at 110.49 45.72 0)
 		(unit 1)
@@
 	)
 	(symbol
-		(lib_id "Device:LED")
+		(lib_id "Library:LED")
 		(at 142.24 105.41 180)
 		(unit 1)
@@
 	)
 	(symbol
-		(lib_id "power:GND")
+		(lib_id "Library:GND")
 		(at 161.29 76.2 0)
 		(unit 1)
@@
 	)
 	(symbol
-		(lib_id "power:GND")
+		(lib_id "Library:GND")
 		(at 179.07 97.79 90)
 		(unit 1)
@@
 	)
 	(symbol
-		(lib_id "Device:C")
+		(lib_id "Library:C")
 		(at 177.8 85.09 0)
 		(unit 1)
@@
 	)
 	(symbol
-		(lib_id "power:+12V")
+		(lib_id "Library:+12V")
 		(at 90.17 46.99 0)
 		(unit 1)
@@
 	)
 	(symbol
-		(lib_id "Regulator_Linear:LM1117DT-5.0")
+		(lib_id "Library:LM1117DT-5.0")
 		(at 100.33 50.8 0)
 		(unit 1)
@@
 	)
 	(symbol
-		(lib_id "power:-12V")
+		(lib_id "Library:-12V")
 		(at 163.83 97.79 90)
 		(unit 1)
@@
 	)
 	(symbol
-		(lib_id "ADP150AUJZ-2.0-R7:ADP150AUJZ-2.0-R7")
+		(lib_id "Library:ADP150AUJZ-2.0-R7")
 		(at 160.02 53.34 0)
 		(unit 1)
@@
 	)
 	(symbol
-		(lib_id "power:-12V")
+		(lib_id "Library:-12V")
 		(at 111.76 83.82 270)
 		(unit 1)
@@
 	)
 	(symbol
-		(lib_id "Device:R")
+		(lib_id "Library:R")
 		(at 134.62 97.79 90)
 		(unit 1)
@@
 	)
 	(symbol
-		(lib_id "Device:C")
+		(lib_id "Library:C")
 		(at 173.99 67.31 0)
 		(mirror y)
