File: effectHardware/f411re.kicad_sch (KiCad schematic)
At the start: 79 parts, among them J1 FTSH-105-XX-X-DV, J3 Conn_02x03_Row_Letter_Last, J4 Conn_01x03, J9 FH12-30S-0.5SH_55_, U2 STM32F411RETx, U5 PEC11L-4015F-S0020, U6 PEC11L-4015F-S0020, U7 74HC14, Y2 MURATA_XRCGB24M000F1SBBR0

Commit message: added lib
Parts:
- C13, C14, C15, C16, C17, C18, C19, C20, C21, C22, C23, C24, C25, C26, C27, C28, C29, C30, C31, C32, C33, C34, C35: symbol Device:C -> Library:C
- C76, C77, C78, C79, C80, C81: symbol Device:C_Small -> Library:C_Small
- D10, D9: symbol Diode:1N4148 -> Library:1N4148
- J1: symbol FTSH-105-XX-X-DV:FTSH-105-XX-X-DV -> Library:FTSH-105-XX-X-DV
- J3: symbol Connector_Generic:Conn_02x03_Row_Letter_Last -> Library:Conn_02x03_Row_Letter_Last
- J4: symbol Connector_Generic:Conn_01x03 -> Library:Conn_01x03
- J9: symbol FH12-30S-0_5SH_55_:FH12-30S-0.5SH_55_ -> Library:FH12-30S-0.5SH_55_
- JP1: symbol Jumper:SolderJumper_2_Open -> Library:SolderJumper_2_Open
- L1: symbol Device:L -> Library:L
- R10, R11, R12, R13, R14, R15, R16, R17, R18, R19, R20, R21, R22, R23, R24, R25, R26, R27, R28, R29, R30, R31, R32, R33, R38, R39, R5, R53, R54, R6, R7, R8, R9: symbol Device:R -> Library:R
- S1, S2, S3, S4: symbol 6425.1101:6425.1101 -> Library:6425.1101
- U2: symbol MCU_ST_STM32F4:STM32F411RETx -> Library:STM32F411RETx
- U5, U6: symbol PEC11L-4015F-S0020:PEC11L-4015F-S0020 -> Library:PEC11L-4015F-S0020
- U7: symbol 74xx:74HC14 -> Library:74HC14
- Y2: symbol MURATA_XRCGB24M000F1SBBR0:MURATA_XRCGB24M000F1SBBR0 -> Library:MURATA_XRCGB24M000F1SBBR0
