File: effectHardware/inputs.kicad_sch (KiCad schematic)
At the start: 86 parts, among them J10 PJ301M-12, J11 PJ301M-12, J12 PJ301M-12, J13 PJ301M-12, J14 PJ301M-12, J15 PJ301M-12, J16 PJ301M-12, J17 PJ301M-12, J18 PJ301M-12, J19 PJ301M-12, J20 PJ301M-12, J5 PJ301M-12, J6 PJ301M-12, J7 PJ301M-12, J8 PJ301M-12, U1 LM4040DCK-10, U10 MCP6004, U11 MCP6004, U8 MCP6004, U9 MCP6004

Commit message: added lib
Parts:
- C36, C37, C38, C39, C40, C42, C43, C44, C45, C46, C47, C48, C49, C50, C51, C52, C53, C54, C55, C56: symbol Device:C -> Library:C
- J10, J11, J12, J13, J14, J15, J16, J17, J18, J19, J20, J5, J6, J7, J8: symbol eurocad:PJ301M-12 -> Library:PJ301M-12
- R40, R41, R42, R43, R44, R45, R46, R47, R48, R49, R50, R51, R52, R55, R56, R57, R58, R59, R60, R62, R63, R64, R65, R66, R67, R68, R69, R70, R71, R72, R73, R74, R75, R76, R77, R78, R79, R80, R81, R82, R83, R84, R85, R86, R87, R88: symbol Device:R -> Library:R
- U1: symbol Reference_Voltage:LM4040DCK-10 -> Library:LM4040DCK-10
- U10, U11, U8, U9: symbol Amplifier_Operational:MCP6004 -> Library:MCP6004
